File: hardware/kicad/ft231x_breakout_usb_power_switch/ft231x_breakout_usb_power_switch.sch (KiCad schematic (older format))
At the start: 51 parts, among them J1 USB_B_Micro_ALT, J2 USB_A_ALT, J3 Conn_01x08, J4 Conn_01x06, J5 Conn_01x08, Q3 2N7002, U1 SRV05-4, U2 FT231XS, U3 TPS2553DBVR, U4 SN74LVC1G04DBVR

Commit message: CI test
Connections:
- net RXLED: no longer JP2.2 (B)
- new net RXLEDD: JP2.2 (B)
Changed lines of the file:
@@
 $EndComp
 Text Label 2650 5200 0    50   ~ 0
-RXLED
+RXLEDD
 Wire Wire Line
 	2300 5700 2250 5700

Commit message: tidy up kibot library warnings
Connections:
- net RXLEDD is gone; now on net RXLED: JP2.2 (B)
Changed lines of the file:
@@
 F 1 "USB_A_ALT" H 9800 1600 50  0000 R CNN
 F 2 "-Connector:TE_292303-1" H 10150 1900 50  0001 C CNN
-F 3 " ~" H 10150 1900 50  0001 C CNN
+F 3 "" H 10150 1900 50  0001 C CNN
 	1    10000 1950
 	-1   0    0    -1
@@
 $EndComp
 Text Label 2650 5200 0    50   ~ 0
-RXLEDD
+RXLED
 Wire Wire Line
 	2300 5700 2250 5700

Commit message: test3
Connections:
- net RXLED: no longer JP2.2 (B)
- new net RXLEDD: JP2.2 (B)
Changed lines of the file:
@@
 $EndComp
 Text Label 2650 5200 0    50   ~ 0
-RXLED
+RXLEDD
 Wire Wire Line
 	2300 5700 2250 5700

Commit message: test4
Connections:
- net RXLEDD is gone; now on net RXLED: JP2.2 (B)
Changed lines of the file:
@@
 $EndComp
 Text Label 2650 5200 0    50   ~ 0
-RXLEDD
+RXLED
 Wire Wire Line
 	2300 5700 2250 5700

Commit message: test5
Other:
- note added: "test"
Changed lines of the file:
@@
 	1    0    0    -1
 $EndComp
+Text Notes 2500 4200 0    50   ~ 0
+test
 $EndSCHEMATC

Commit message: test6
Other:
- note added: "test1"
- note removed: "test"
Changed lines of the file:
@@
 $EndComp
 Text Notes 2500 4200 0    50   ~ 0
-test
+test1
 $EndSCHEMATC

Commit message: test7
Other:
- note added: "test7"
- note removed: "test1"
Changed lines of the file:
@@
 $EndComp
 Text Notes 2500 4200 0    50   ~ 0
-test1
+test7
 $EndSCHEMATC

Commit message: test8
Other:
- note added: "test6"
- note removed: "test7"
Changed lines of the file:
@@
 $EndComp
 Text Notes 2500 4200 0    50   ~ 0
-test7
+test6
 $EndSCHEMATC
