File: hardware/kicad/ft231x_breakout_usb_power_switch/ft231x_breakout_usb_power_switch.sch (KiCad schematic (older format))
At the start: 51 parts, among them J1 USB_B_Micro_ALT, J2 USB_A_ALT, J3 Conn_01x08, J4 Conn_01x06, J5 Conn_01x08, Q3 2N7002, U1 SRV05-4, U2 FT231XS, U3 TPS2553DBVR, U4 SN74LVC1G04DBVR

Commit message: change footprint FT231XS to fix lcsc rotation filter
Parts:
- U2: footprint -Chip:FT231XS -> -Chip:SSOP-20_3.9x8.7mm_P0.635mm; element14# (none) -> 2081328; mouser# (none) -> 895-FT231XS-R
Changed lines of the file:
@@
 F 0 "U2" H 5850 3200 50  0000 C CNN
 F 1 "FT231XS" H 6750 1500 50  0000 C CNN
-F 2 "-Chip:FT231XS" H 7350 1600 50  0001 C CNN
+F 2 "-Chip:SSOP-20_3.9x8.7mm_P0.635mm" H 7350 1600 50  0001 C CNN
 F 3 "https://www.ftdichip.com/Support/Documents/DataSheets/ICs/DS_FT231X.pdf" H 6350 2400 50  0001 C CNN
 F 4 "USB to UART USB 2.0 UART Interface 20-SSOP" H 6350 2400 50  0001 C CNN "Desc"
@@
 F 7 "C132160" H 6350 2400 50  0001 C CNN "LCSC#"
 F 8 "768-1129-2-ND" H 6350 2400 50  0001 C CNN "digikey#"
+F 9 "2081328" H 6350 2400 50  0001 C CNN "element14#"
+F 10 "895-FT231XS-R" H 6350 2400 50  0001 C CNN "mouser#"
 	1    6350 2400
 	1    0    0    -1
@@
 F 0 "PCB1" H 7550 6416 40  0000 C CNN
 F 1 "PCB - 2 Layer" H 7550 6300 30  0001 C CNN
-F 2 "" H 7550 6200 60  0000 C CNN
+F 2 "" H 7550 6200 60  0001 C CNN
 F 3 "" H 7550 6200 60  0000 C CNN
 	1    7550 6300

Commit message: Add substitute field
Parts:
- U2: substitute (none) -> No
Changed lines of the file:
@@
 F 5 "FTDI" H 6350 2400 50  0001 C CNN "manf"
 F 6 "FT231XS-R" H 6350 2400 50  0001 C CNN "manf#"
-F 7 "C132160" H 6350 2400 50  0001 C CNN "LCSC#"
-F 8 "768-1129-2-ND" H 6350 2400 50  0001 C CNN "digikey#"
-F 9 "2081328" H 6350 2400 50  0001 C CNN "element14#"
-F 10 "895-FT231XS-R" H 6350 2400 50  0001 C CNN "mouser#"
+F 7 "No" H 6350 2400 50  0001 C CNN "substitute"
+F 8 "C132160" H 6350 2400 50  0001 C CNN "LCSC#"
+F 9 "768-1129-2-ND" H 6350 2400 50  0001 C CNN "digikey#"
+F 10 "2081328" H 6350 2400 50  0001 C CNN "element14#"
+F 11 "895-FT231XS-R" H 6350 2400 50  0001 C CNN "mouser#"
 	1    6350 2400
 	1    0    0    -1

Commit message: Add value to kibot kibom grouping
Parts:
- C1: Desc (none) -> 100nF ±10% 50V X7R 0603 Multilayer Ceramic Capacitors MLCC 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; LCSC# (none) -> C14663; digikey# (none) -> 311-1344-1-ND; element14# (none) -> 1362556; manf (none) -> Yageo; manf# (none) -> CC0603KRX7R9BB104; mouser# (none) -> 603-CC603KRX7R9BB104; substitute (none) -> Yes
- C3: Des (none) -> 100nF ±10% 50V X7R 0603 Multilayer Ceramic Capacitors MLCC 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; LCSC# (none) -> C14663; digikey# (none) -> 311-1344-1-ND; element14# (none) -> 1362556; manf (none) -> Yageo; manf# (none) -> CC0603KRX7R9BB104; mouser# (none) -> 603-CC603KRX7R9BB104; substitute (none) -> Yes
Changed lines of the file:
@@
 F 0 "C1" H 1100 3350 50  0000 L CNN
 F 1 "0.1uF" H 950 3150 50  0000 L CNN
-F 2 "-Passive:C_0603" H 1238 3100 50  0001 C CNN
-F 3 "" H 1200 3250 50  0001 C CNN
+F 2 "-Passive:C_0603" H 1238 3100 50  0001 L CNN
+F 3 "https://www.yageo.com/upload/media/product/productsearch/datasheet/mlcc/UPY-GPHC_X7R_6.3V-to-50V_20.pdf" H 1200 3250 50  0001 L CNN
+F 4 "100nF ±10% 50V X7R 0603 Multilayer Ceramic Capacitors MLCC - SMD/SMT RoHS" H 1200 3250 50  0001 L CNN "Desc"
+F 5 "Yageo" H 1200 3250 50  0001 L CNN "manf"
+F 6 "CC0603KRX7R9BB104" H 1200 3250 50  0001 L CNN "manf#"
+F 7 "Yes" H 1200 3250 50  0001 L CNN "substitute"
+F 8 "C14663" H 1200 3250 50  0001 L CNN "LCSC#"
+F 9 "311-1344-1-ND" H 1200 3250 50  0001 L CNN "digikey#"
+F 10 "1362556" H 1200 3250 50  0001 L CNN "element14#"
+F 11 "603-CC603KRX7R9BB104" H 1200 3250 50  0001 L CNN "mouser#"
 	1    1200 3250
 	1    0    0    -1
@@
 F 1 "0.1uF" H 3550 3150 50  0000 L CNN
 F 2 "-Passive:C_0603" H 3838 3100 50  0001 C CNN
-F 3 "" H 3800 3250 50  0001 C CNN
+F 3 "https://www.yageo.com/upload/media/product/productsearch/datasheet/mlcc/UPY-GPHC_X7R_6.3V-to-50V_20.pdf" H 3800 3250 50  0001 C CNN
+F 4 "100nF ±10% 50V X7R 0603 Multilayer Ceramic Capacitors MLCC - SMD/SMT RoHS" H 3800 3250 50  0001 C CNN "Des"
+F 5 "Yageo" H 3800 3250 50  0001 C CNN "manf"
+F 6 "CC0603KRX7R9BB104" H 3800 3250 50  0001 C CNN "manf#"
+F 7 "Yes" H 3800 3250 50  0001 C CNN "substitute"
+F 8 "C14663" H 3800 3250 50  0001 C CNN "LCSC#"
+F 9 "311-1344-1-ND" H 3800 3250 50  0001 C CNN "digikey#"
+F 10 "1362556" H 3800 3250 50  0001 C CNN "element14#"
+F 11 "603-CC603KRX7R9BB104" H 3800 3250 50  0001 C CNN "mouser#"
 	1    3800 3250
 	1    0    0    -1

Commit message: bom fields for 0.1uF caps
Parts:
- C10, C11, C7, C8: Desc (none) -> 100nF ±10% 50V X7R 0603 Multilayer Ceramic Capacitors MLCC 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; LCSC# (none) -> C14663; digikey# (none) -> 311-1344-1-ND; element14# (none) -> 1362556; manf (none) -> Yageo; manf# (none) -> CC0603KRX7R9BB104; mouser# (none) -> 603-CC603KRX7R9BB104; substitute (none) -> Yes
Changed lines of the file:
@@
 F 0 "C7" H 5100 3350 50  0000 L CNN
 F 1 "0.1uF" H 5050 3150 50  0000 L CNN
-F 2 "-Passive:C_0603" H 5338 3100 50  0001 C CNN
-F 3 "" H 5300 3250 50  0001 C CNN
+F 2 "-Passive:C_0603" H 5338 3100 50  0001 L CNN
+F 3 "https://www.yageo.com/upload/media/product/productsearch/datasheet/mlcc/UPY-GPHC_X7R_6.3V-to-50V_20.pdf" H 5300 3250 50  0001 L CNN
+F 4 "100nF ±10% 50V X7R 0603 Multilayer Ceramic Capacitors MLCC - SMD/SMT RoHS" H 5300 3250 50  0001 L CNN "Desc"
+F 5 "Yageo" H 5300 3250 50  0001 L CNN "manf"
+F 6 "CC0603KRX7R9BB104" H 5300 3250 50  0001 L CNN "manf#"
+F 7 "Yes" H 5300 3250 50  0001 L CNN "substitute"
+F 8 "C14663" H 5300 3250 50  0001 L CNN "LCSC#"
+F 9 "311-1344-1-ND" H 5300 3250 50  0001 L CNN "digikey#"
+F 10 "1362556" H 5300 3250 50  0001 L CNN "element14#"
+F 11 "603-CC603KRX7R9BB104" H 5300 3250 50  0001 L CNN "mouser#"
 	1    5300 3250
 	1    0    0    -1
@@
 F 0 "C8" H 8100 3350 50  0000 L CNN
 F 1 "0.1uF" H 8100 3150 50  0000 L CNN
-F 2 "-Passive:C_0603" H 8138 3100 50  0001 C CNN
-F 3 "" H 8100 3250 50  0001 C CNN
+F 2 "-Passive:C_0603" H 8138 3100 50  0001 L CNN
+F 3 "https://www.yageo.com/upload/media/product/productsearch/datasheet/mlcc/UPY-GPHC_X7R_6.3V-to-50V_20.pdf" H 8100 3250 50  0001 L CNN
+F 4 "100nF ±10% 50V X7R 0603 Multilayer Ceramic Capacitors MLCC - SMD/SMT RoHS" H 8100 3250 50  0001 L CNN "Desc"
+F 5 "Yageo" H 8100 3250 50  0001 L CNN "manf"
+F 6 "CC0603KRX7R9BB104" H 8100 3250 50  0001 L CNN "manf#"
+F 7 "Yes" H 8100 3250 50  0001 L CNN "substitute"
+F 8 "C14663" H 8100 3250 50  0001 L CNN "LCSC#"
+F 9 "311-1344-1-ND" H 8100 3250 50  0001 L CNN "digikey#"
+F 10 "1362556" H 8100 3250 50  0001 L CNN "element14#"
+F 11 "603-CC603KRX7R9BB104" H 8100 3250 50  0001 L CNN "mouser#"
 	1    8100 3250
 	1    0    0    -1
@@
 F 0 "C10" H 900 7200 50  0000 L CNN
 F 1 "0.1uF" H 900 7000 50  0000 L CNN
-F 2 "-Passive:C_0603" H 938 6950 50  0001 C CNN
-F 3 "" H 900 7100 50  0001 C CNN
+F 2 "-Passive:C_0603" H 938 6950 50  0001 L CNN
+F 3 "https://www.yageo.com/upload/media/product/productsearch/datasheet/mlcc/UPY-GPHC_X7R_6.3V-to-50V_20.pdf" H 900 7100 50  0001 L CNN
+F 4 "100nF ±10% 50V X7R 0603 Multilayer Ceramic Capacitors MLCC - SMD/SMT RoHS" H 900 7100 50  0001 R CNN "Desc"
+F 5 "Yageo" H 900 7100 50  0001 L CNN "manf"
+F 6 "CC0603KRX7R9BB104" H 900 7100 50  0001 L CNN "manf#"
+F 7 "Yes" H 900 7100 50  0001 L CNN "substitute"
+F 8 "C14663" H 900 7100 50  0001 L CNN "LCSC#"
+F 9 "311-1344-1-ND" H 900 7100 50  0001 L CNN "digikey#"
+F 10 "1362556" H 900 7100 50  0001 L CNN "element14#"
+F 11 "603-CC603KRX7R9BB104" H 900 7100 50  0001 L CNN "mouser#"
 	1    900  7100
 	1    0    0    -1
@@
 F 0 "C11" H 10450 3350 50  0000 L CNN
 F 1 "0.1uF" H 10450 3150 50  0000 L CNN
-F 2 "-Passive:C_0603" H 10488 3100 50  0001 C CNN
-F 3 "" H 10450 3250 50  0001 C CNN
+F 2 "-Passive:C_0603" H 10488 3100 50  0001 L CNN
+F 3 "https://www.yageo.com/upload/media/product/productsearch/datasheet/mlcc/UPY-GPHC_X7R_6.3V-to-50V_20.pdf" H 10450 3250 50  0001 L CNN
+F 4 "100nF ±10% 50V X7R 0603 Multilayer Ceramic Capacitors MLCC - SMD/SMT RoHS" H 10450 3250 50  0001 L CNN "Desc"
+F 5 "Yageo" H 10450 3250 50  0001 L CNN "manf"
+F 6 "CC0603KRX7R9BB104" H 10450 3250 50  0001 L CNN "manf#"
+F 7 "Yes" H 10450 3250 50  0001 L CNN "substitute"
+F 8 "C14663" H 10450 3250 50  0001 L CNN "LCSC#"
+F 9 "311-1344-1-ND" H 10450 3250 50  0001 L CNN "digikey#"
+F 10 "1362556" H 10450 3250 50  0001 L CNN "element14#"
+F 11 "603-CC603KRX7R9BB104" H 10450 3250 50  0001 L CNN "mouser#"
 	1    10450 3250
 	1    0    0    -1

Commit message: 10nF cap BOM fields
Parts:
- C2: Desc (none) -> 10nF ±10% 50V X7R 0603 Multilayer Ceramic Capacitors MLCC -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; LCSC# (none) -> C100042; digikey# (none) -> 311-1085-2-ND; element14# (none) -> 722236; manf (none) -> Yageo; manf# (none) -> CC0603KRX7R9BB103; mouser# (none) -> 603-CC603KRX7R9BB103; substitute (none) -> Yes
Changed lines of the file:
@@
 F 0 "C2" H 3250 3350 50  0000 L CNN
 F 1 "10nF" H 3200 3150 50  0000 L CNN
-F 2 "-Passive:C_0603" H 3438 3100 50  0001 C CNN
-F 3 "" H 3400 3250 50  0001 C CNN
+F 2 "-Passive:C_0603" H 3438 3100 50  0001 L CNN
+F 3 "https://www.yageo.com/upload/media/product/productsearch/datasheet/mlcc/UPY-GPHC_X7R_6.3V-to-50V_20.pdf" H 3400 3250 50  0001 L CNN
+F 4 "10nF ±10% 50V X7R 0603 Multilayer Ceramic Capacitors MLCC - SMD/SMT RoHS" H 3400 3250 50  0001 L CNN "Desc"
+F 5 "Yageo" H 3400 3250 50  0001 L CNN "manf"
+F 6 "CC0603KRX7R9BB103" H 3400 3250 50  0001 L CNN "manf#"
+F 7 "Yes" H 3400 3250 50  0001 L CNN "substitute"
+F 8 "C100042" H 3400 3250 50  0001 L CNN "LCSC#"
+F 9 "311-1085-2-ND" H 3400 3250 50  0001 L CNN "digikey#"
+F 10 "722236" H 3400 3250 50  0001 L CNN "element14#"
+F 11 "603-CC603KRX7R9BB103" H 3400 3250 50  0001 L CNN "mouser#"
 	1    3400 3250
 	1    0    0    -1

Commit message: BOM fields 47 pF cap
Parts:
- C5, C6: Desc (none) -> 47pF ±5% 50V NP0 0603 Multilayer Ceramic Capacitors MLCC - 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; LCSC# (none) -> C105622; digikey# (none) -> 311-1065-1-ND; element14# (none) -> 722042; manf (none) -> Yageo; manf# (none) -> CC0603JRNPO9BN470; mouser# (none) -> 603-CC603JRNPO9BN470; substitute (none) -> Yes
Changed lines of the file:
@@
 F 0 "C6" H 4800 3350 50  0000 L CNN
 F 1 "47pF" H 4800 3150 50  0000 L CNN
-F 2 "-Passive:C_0603" H 4838 3100 50  0001 C CNN
-F 3 "" H 4800 3250 50  0001 C CNN
+F 2 "-Passive:C_0603" H 4838 3100 50  0001 L CNN
+F 3 "https://www.yageo.com/upload/media/product/productsearch/datasheet/mlcc/UPY-GP_NP0_16V-to-50V_18.pdf" H 4800 3250 50  0001 L CNN
+F 4 "47pF ±5% 50V NP0 0603 Multilayer Ceramic Capacitors MLCC - SMD/SMT RoHS" H 4800 3250 50  0001 L CNN "Desc"
+F 5 "Yageo" H 4800 3250 50  0001 L CNN "manf"
+F 6 "CC0603JRNPO9BN470" H 4800 3250 50  0001 L CNN "manf#"
+F 7 "Yes" H 4800 3250 50  0001 L CNN "substitute"
+F 8 "C105622" H 4800 3250 50  0001 L CNN "LCSC#"
+F 9 "311-1065-1-ND" H 4800 3250 50  0001 L CNN "digikey#"
+F 10 "722042" H 4800 3250 50  0001 L CNN "element14#"
+F 11 "603-CC603JRNPO9BN470" H 4800 3250 50  0001 L CNN "mouser#"
 	1    4800 3250
 	1    0    0    -1
@@
 F 0 "C5" H 4550 3350 50  0000 L CNN
 F 1 "47pF" H 4550 3150 50  0000 L CNN
-F 2 "-Passive:C_0603" H 4588 3100 50  0001 C CNN
-F 3 "" H 4550 3250 50  0001 C CNN
+F 2 "-Passive:C_0603" H 4588 3100 50  0001 L CNN
+F 3 "https://www.yageo.com/upload/media/product/productsearch/datasheet/mlcc/UPY-GP_NP0_16V-to-50V_18.pdf" H 4550 3250 50  0001 L CNN
+F 4 "47pF ±5% 50V NP0 0603 Multilayer Ceramic Capacitors MLCC - SMD/SMT RoHS" H 4550 3250 50  0001 L CNN "Desc"
+F 5 "Yageo" H 4550 3250 50  0001 L CNN "manf"
+F 6 "CC0603JRNPO9BN470" H 4550 3250 50  0001 L CNN "manf#"
+F 7 "Yes" H 4550 3250 50  0001 L CNN "substitute"
+F 8 "C105622" H 4550 3250 50  0001 L CNN "LCSC#"
+F 9 "311-1065-1-ND" H 4550 3250 50  0001 L CNN "digikey#"
+F 10 "722042" H 4550 3250 50  0001 L CNN "element14#"
+F 11 "603-CC603JRNPO9BN470" H 4550 3250 50  0001 L CNN "mouser#"
 	1    4550 3250
 	1    0    0    -1

Commit message: 4.7 uF BOM fields
Parts:
- C4: Desc (none) -> 4.7uF ±10% 10V X5R 0603 Multilayer Ceramic Capacitors MLCC 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; LCSC# (none) -> C109456; digikey# (none) -> 311-1455-1-ND; element14# (none) -> 1458898; manf (none) -> Yageo; manf# (none) -> CC0603KRX5R6BB475; mouser# (none) -> 603-CC603KRX5R6BB475; substitute (none) -> Yes
Changed lines of the file:
@@
 F 0 "C4" H 4000 3350 50  0000 L CNN
 F 1 "4.7uF" H 3900 3150 50  0000 L CNN
-F 2 "-Passive:C_0603" H 4188 3100 50  0001 C CNN
-F 3 "" H 4150 3250 50  0001 C CNN
+F 2 "-Passive:C_0603" H 4188 3100 50  0001 L CNN
+F 3 "https://www.yageo.com/upload/media/product/productsearch/datasheet/mlcc/UPY-GPHC_X5R_4V-to-50V_26.pdf" H 4150 3250 50  0001 L CNN
+F 4 "4.7uF ±10% 10V X5R 0603 Multilayer Ceramic Capacitors MLCC - SMD/SMT RoHS" H 4150 3250 50  0001 L CNN "Desc"
+F 5 "Yageo" H 4150 3250 50  0001 L CNN "manf"
+F 6 "CC0603KRX5R6BB475" H 4150 3250 50  0001 L CNN "manf#"
+F 7 "Yes" H 4150 3250 50  0001 L CNN "substitute"
+F 8 "C109456" H 4150 3250 50  0001 L CNN "LCSC#"
+F 9 "311-1455-1-ND" H 4150 3250 50  0001 L CNN "digikey#"
+F 10 "1458898" H 4150 3250 50  0001 L CNN "element14#"
+F 11 "603-CC603KRX5R6BB475" H 4150 3250 50  0001 L CNN "mouser#"
 	1    4150 3250
 	1    0    0    -1

Commit message: 150 uF cap bom fields
Parts:
- C9: Desc (none) -> 150uF ±20% 6.3V 25 mΩ @ 100kHz -55℃ ~ +105℃ CASE-B_3528 Tan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; LCSC# (none) -> C156458; digikey# (none) -> 399-5753-1-ND; element14# (none) -> 2491063; manf (none) -> KEMET; manf# (none) -> T520B157M006ATE025; mouser# (none) -> 80-T520B157M006ATE25; substitute (none) -> Yes
Changed lines of the file:
@@
 F 0 "C9" H 9665 3296 50  0000 L CNN
 F 1 "150uF" H 9665 3205 50  0000 L CNN
-F 2 "-Discrete:EIA-3528-12_Kemet-T_DENSITY_MEDIUM" H 9550 3250 50  0001 C CNN
-F 3 "" H 9550 3250 50  0001 C CNN
+F 2 "-Discrete:EIA-3528-12_Kemet-T_DENSITY_MEDIUM" H 9550 3250 50  0001 L CNN
+F 3 "https://api.kemet.com/component-edge/download/datasheet/T520B157M006ATE025.pdf" H 9550 3250 50  0001 L CNN
+F 4 "150uF ±20% 6.3V 25 mΩ @ 100kHz -55℃ ~ +105℃ CASE-B_3528 Tantalum Capacitors RoHS" H 9550 3250 50  0001 L CNN "Desc"
+F 5 "KEMET" H 9550 3250 50  0001 L CNN "manf"
+F 6 "T520B157M006ATE025" H 9550 3250 50  0001 L CNN "manf#"
+F 7 "Yes" H 9550 3250 50  0001 L CNN "substitute"
+F 8 "C156458" H 9550 3250 50  0001 L CNN "LCSC#"
+F 9 "399-5753-1-ND" H 9550 3250 50  0001 L CNN "digikey#"
+F 10 "2491063" H 9550 3250 50  0001 L CNN "element14#"
+F 11 "80-T520B157M006ATE25" H 9550 3250 50  0001 L CNN "mouser#"
 	1    9550 3250
 	1    0    0    -1
