File: hardware/kicad/ft231x_breakout_usb_power_switch/ft231x_breakout_usb_power_switch.sch (KiCad schematic (older format))
At the start: 51 parts, among them J1 USB_B_Micro_ALT, J2 USB_A_ALT, J3 Conn_01x08, J4 Conn_01x06, J5 Conn_01x08, Q3 2N7002, U1 SRV05-4, U2 FT231XS, U3 TPS2553DBVR, U4 SN74LVC1G04DBVR

Commit message: reset switch initial
Parts:
- added C12: 0.1uF, -Passive:C_0603, symbol -Passive:C
- added R14: 1k, -Passive:R_0603, symbol -Passive:R
- added SW1: SW_MEC_5G, -Switch:B3U-1000P, symbol -Switch:SW_MEC_5G
Connections:
- wire segments 179 -> 187
Other:
- note added: "Micro USB\nInput"
- note removed: "Micro USB Input"
- moved on the sheet: C1, C11, C2, C3, C4, C5, C6, C7, C8, C9, FB1, J1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

Commit message: add optional pull down to enable
Parts:
- added C13, C14: 0.1uF, -Passive:C_0603, symbol -Passive:C
- added JP8: SolderJumper_2_Bridged_Alt, -Jumper:SolderJumper-2_P1.3mm_Un-Bridged_RoundedPad1.0x1.5mm, symbol -Jumper:SolderJumper_2_Bridged_Alt
- added R15: 1k, -Passive:R_0603, symbol -Passive:R
- added U5, U6: NC7SZ66M5X, -Chip:SOT-23-5, symbol -Chip:NC7SZ66M5X
- SW1: value SW_MEC_5G -> B3U-1000P; Desc (none) -> Tactile Switch SPST-NO Top Actuated Surface Mount; LCSC# (none) -> C231329; digikey# (none) -> SW1020CT-ND; element14# (none) -> 1333652; manf (none) -> Omron Electronics; manf# (none) -> B3U-1000P; mouser# (none) -> 653-B3U-1000P
Connections:
- net labels added: EN, RES, SRES, STXD
- net labels removed: ENLED, RESET
- wire segments 187 -> 210
Other:
- note added: "Bus Switch (To Prevent Back Powering Target Over UART)"
- note added: "USB power output is enabled by\ndefault. To disable USB output\non power up, bridge jumper JP8."
- moved on the sheet: C1, C10, C11, C12, C2, C3, C4, C5, C6, C7, C8, C9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

Commit message: Reset switch and bus switches routed
Parts:
- added R16, R17: 1k, -Passive:R_0603, symbol -Passive:R
Connections:
- wire segments 210 -> 212
Other:
- moved on the sheet: C10, C13, C14, D4, JP7, R11

Commit message: Fix reset when FT231X is drivng power switch OE
Parts:
- added R18: 10k, -Passive:R_0603, symbol -Passive:R
Connections:
- wire segments 212 -> 213
Other:
- moved on the sheet: JP8, R15
Changed lines of the file:
@@
 	0    -1   -1   0
 $EndComp
-Text Label 7750 2350 2    50   ~ 0
+Text Label 7800 2350 2    50   ~ 0
 EN
 Text Label 1450 6050 2    50   ~ 0
@@
 U 1 1 6114CC1F
 P 8100 2050
-F 0 "R12" V 8200 2050 50  0000 C CNN
+F 0 "R12" H 7950 2050 50  0000 C CNN
 F 1 "1k" V 8100 2050 50  0000 C CNN
 F 2 "-Passive:R_0603" V 8030 2050 50  0001 C CNN
@@
 	5350 1450 4950 1450
 Wire Wire Line
-	8100 2350 8100 2200
-Wire Wire Line
 	8100 1900 8100 1750
 Wire Wire Line
@@
 	950  3050 950  2950
 Connection ~ 1100 3050
-Connection ~ 8100 2350
 Wire Wire Line
 	1250 1750 1250 2550
@@
 Wire Wire Line
 	10150 2550 10150 2650
-Wire Wire Line
-	8100 2350 8100 2550
 Wire Wire Line
 	8050 2550 8100 2550
@@
 L -Passive:R R15
 U 1 1 60FED1B8
-P 7400 2900
-F 0 "R15" H 7550 2900 50  0000 C CNN
-F 1 "1k" V 7400 2900 50  0000 C CNN
-F 2 "-Passive:R_0603" V 7330 2900 50  0001 C CNN
-F 3 "https://www.yageo.com/upload/media/product/productsearch/datasheet/rchip/PYu-RC_Group_51_RoHS_L_11.pdf" H 7400 2900 50  0001 C CNN
-F 4 "1kΩ ±5% 0.1W ±100ppm/℃ 0603 Chip Resistor - Surface Mount RoHS" H 7400 2900 50  0001 C CNN "Desc"
-F 5 "Yageo" H 7400 2900 50  0001 C CNN "manf"
-F 6 "RC0603JR-071KL" H 7400 2900 50  0001 C CNN "manf#"
-F 7 "Yes" H 7400 2900 50  0001 C CNN "substitute"
-F 8 "C14676" H 7400 2900 50  0001 C CNN "LCSC#"
-F 9 "311-1.0KGRTR-ND" H 7400 2900 50  0001 C CNN "digikey#"
-F 10 "9233385" H 7400 2900 50  0001 C CNN "element14#"
-F 11 "603-RC0603JR-071KL" H 7400 2900 50  0001 C CNN "mouser#"
-	1    7400 2900
+P 8500 2900
+F 0 "R15" H 8350 2900 50  0000 C CNN
+F 1 "1k" V 8500 2900 50  0000 C CNN
+F 2 "-Passive:R_0603" V 8430 2900 50  0001 C CNN
+F 3 "https://www.yageo.com/upload/media/product/productsearch/datasheet/rchip/PYu-RC_Group_51_RoHS_L_11.pdf" H 8500 2900 50  0001 C CNN
+F 4 "1kΩ ±5% 0.1W ±100ppm/℃ 0603 Chip Resistor - Surface Mount RoHS" H 8500 2900 50  0001 C CNN "Desc"
+F 5 "Yageo" H 8500 2900 50  0001 C CNN "manf"
+F 6 "RC0603JR-071KL" H 8500 2900 50  0001 C CNN "manf#"
+F 7 "Yes" H 8500 2900 50  0001 C CNN "substitute"
+F 8 "C14676" H 8500 2900 50  0001 C CNN "LCSC#"
+F 9 "311-1.0KGRTR-ND" H 8500 2900 50  0001 C CNN "digikey#"
+F 10 "9233385" H 8500 2900 50  0001 C CNN "element14#"
+F 11 "603-RC0603JR-071KL" H 8500 2900 50  0001 C CNN "mouser#"
+	1    8500 2900
 	-1   0    0    1
 $EndComp
@@
 L -Jumper:SolderJumper_2_Bridged_Alt JP8
 U 1 1 60FEF385
-P 7400 2550
-F 0 "JP8" V 7400 2400 50  0000 C CNN
-F 1 "SolderJumper_2_Bridged_Alt" V 7445 2618 50  0001 L CNN
-F 2 "-Jumper:SolderJumper-2_P1.3mm_Un-Bridged_RoundedPad1.0x1.5mm" H 7375 2550 50  0001 L CNN
-F 3 "" H 7375 2550 50  0001 L CNN
-F 4 "Solder Jumper Bridged" H 7400 2550 50  0001 L CNN "Desc"
-F 5 "N/A" H 7400 2550 50  0001 L CNN "manf"
-F 6 "N/A" H 7400 2550 50  0001 L CNN "manf#"
-F 7 "No" H 7400 2550 50  0001 L CNN "substitute"
-F 8 "" H 7400 2550 50  0001 L CNN "LCSC#"
-F 9 "" H 7400 2550 50  0001 L CNN "digikey#"
-F 10 "" H 7400 2550 50  0001 L CNN "element14#"
-F 11 "" H 7400 2550 50  0001 L CNN "mouser#"
-	1    7400 2550
+P 8500 2550
+F 0 "JP8" V 8500 2700 50  0000 C CNN
+F 1 "SolderJumper_2_Bridged_Alt" V 8545 2618 50  0001 L CNN
+F 2 "-Jumper:SolderJumper-2_P1.3mm_Un-Bridged_RoundedPad1.0x1.5mm" H 8475 2550 50  0001 L CNN
+F 3 "" H 8475 2550 50  0001 L CNN
+F 4 "Solder Jumper Bridged" H 8500 2550 50  0001 L CNN "Desc"
+F 5 "N/A" H 8500 2550 50  0001 L CNN "manf"
+F 6 "N/A" H 8500 2550 50  0001 L CNN "manf#"
+F 7 "No" H 8500 2550 50  0001 L CNN "substitute"
+F 8 "" H 8500 2550 50  0001 L CNN "LCSC#"
+F 9 "" H 8500 2550 50  0001 L CNN "digikey#"
+F 10 "" H 8500 2550 50  0001 L CNN "element14#"
+F 11 "" H 8500 2550 50  0001 L CNN "mouser#"
+	1    8500 2550
 	0    1    1    0
 $EndComp
@@
 L -Flag:GND #PWR022
 U 1 1 60FF6EA7
-P 7400 3100
-F 0 "#PWR022" H 7400 2850 50  0001 C CNN
-F 1 "GND" H 7400 2950 50  0000 C CNN
-F 2 "" H 7400 3100 50  0001 C CNN
-F 3 "" H 7400 3100 50  0001 C CNN
-	1    7400 3100
-	1    0    0    -1
-$EndComp
-Wire Wire Line
-	7350 2350 7400 2350
-Wire Wire Line
-	7400 2400 7400 2350
-Connection ~ 7400 2350
-Wire Wire Line
-	7400 2350 8100 2350
-Wire Wire Line
-	7400 2750 7400 2700
-Wire Wire Line
-	7400 3100 7400 3050
+P 8500 3100
+F 0 "#PWR022" H 8500 2850 50  0001 C CNN
+F 1 "GND" H 8500 2950 50  0000 C CNN
+F 2 "" H 8500 3100 50  0001 C CNN
+F 3 "" H 8500 3100 50  0001 C CNN
+	1    8500 3100
+	1    0    0    -1
+$EndComp
+Wire Wire Line
+	8500 2750 8500 2700
+Wire Wire Line
+	8500 3100 8500 3050
 Text Notes 5500 3050 0    61   ~ 0
 USB power output is enabled by\ndefault. To disable USB output\non power up, bridge jumper JP8.
@@
 Wire Wire Line
 	7300 5750 7250 5750
+$Comp
+L -Passive:R R18
+U 1 1 6044ADBA
+P 7550 2350
+F 0 "R18" V 7450 2350 50  0000 C CNN
+F 1 "10k" V 7550 2350 50  0000 C CNN
+F 2 "-Passive:R_0603" V 7480 2350 50  0001 L CNN
+F 3 "https://www.yageo.com/upload/media/product/productsearch/datasheet/rchip/PYu-RC_Group_51_RoHS_L_11.pdf" H 7550 2350 50  0001 L CNN
+F 4 "10kΩ ±5% 0.1W ±100ppm/℃ 0603 Chip Resistor - Surface Mount RoHS" H 7550 2350 50  0001 L CNN "Desc"
+F 5 "Yageo" H 7550 2350 50  0001 L CNN "manf"
+F 6 "RC0603JR-0710KL" H 7550 2350 50  0001 L CNN "manf#"
+F 7 "Yes" H 7550 2350 50  0001 L CNN "substitute"
+F 8 "C99198" H 7550 2350 50  0001 L CNN "LCSC#"
+F 9 "311-10KGRTR-ND" H 7550 2350 50  0001 L CNN "digikey#"
+F 10 "9233504" H 7550 2350 50  0001 L CNN "element14#"
+F 11 "603-RC0603JR-0710KL" H 7550 2350 50  0001 L CNN "mouser#"
+	1    7550 2350
+	0    1    1    0
+$EndComp
+Wire Wire Line
+	8100 2200 8100 2350
+Wire Wire Line
+	7700 2350 8100 2350
+Connection ~ 8100 2350
+Wire Wire Line
+	8100 2350 8100 2550
+Wire Wire Line
+	7350 2350 7400 2350
+Wire Wire Line
+	8500 2400 8500 2350
+Wire Wire Line
+	8500 2350 8100 2350
 $EndSCHEMATC

Commit message: Add two fiducials
Parts:
- added FID1, FID2: Fiducial, -Mechanical:Fiducial_1mm_Mask2mm, symbol -Mechanical:Fiducial
Other:
- moved on the sheet: PCB1
Changed lines of the file:
@@
 L -Module:PCB PCB1
 U 1 1 602766F4
-P 5350 7300
-F 0 "PCB1" H 5350 7416 40  0000 C CNN
-F 1 "PCB - 2 Layer" H 5350 7300 30  0000 C CNN
-F 2 "" H 5350 7200 60  0001 L CNN
-F 3 "" H 5350 7200 60  0001 L CNN
-F 4 "PCB, 2 Layer 1.6mm, 1.0 oz Copper, Green Soldermask, White Silkscreen, ENIG,  RoHs" H 5350 7300 50  0001 L CNN "Desc"
-F 5 "N/A" H 5350 7300 50  0001 L CNN "manf"
-F 6 "N/A" H 5350 7300 50  0001 L CNN "manf#"
-F 7 "No" H 5350 7300 50  0001 L CNN "substitute"
-F 8 "" H 5350 7300 50  0001 L CNN "LCSC#"
-F 9 "" H 5350 7300 50  0001 L CNN "digikey#"
-F 10 "" H 5350 7300 50  0001 L CNN "element14#"
-F 11 "" H 5350 7300 50  0001 L CNN "mouser#"
-	1    5350 7300
+P 4800 7300
+F 0 "PCB1" H 4800 7416 40  0000 C CNN
+F 1 "PCB - 2 Layer" H 4800 7300 30  0000 C CNN
+F 2 "" H 4800 7200 60  0001 L CNN
+F 3 "" H 4800 7200 60  0001 L CNN
+F 4 "PCB, 2 Layer 1.6mm, 1.0 oz Copper, Green Soldermask, White Silkscreen, ENIG,  RoHs" H 4800 7300 50  0001 L CNN "Desc"
+F 5 "N/A" H 4800 7300 50  0001 L CNN "manf"
+F 6 "N/A" H 4800 7300 50  0001 L CNN "manf#"
+F 7 "No" H 4800 7300 50  0001 L CNN "substitute"
+F 8 "" H 4800 7300 50  0001 L CNN "LCSC#"
+F 9 "" H 4800 7300 50  0001 L CNN "digikey#"
+F 10 "" H 4800 7300 50  0001 L CNN "element14#"
+F 11 "" H 4800 7300 50  0001 L CNN "mouser#"
+	1    4800 7300
 	1    0    0    -1
 $EndComp
@@
 Wire Wire Line
 	8500 2350 8100 2350
+$Comp
+L -Mechanical:Fiducial FID1
+U 1 1 6051AB3D
+P 5350 7250
+F 0 "FID1" H 5435 7296 50  0000 L CNN
+F 1 "Fiducial" H 5435 7205 50  0000 L CNN
+F 2 "-Mechanical:Fiducial_1mm_Mask2mm" H 5350 7250 50  0001 C CNN
+F 3 "~" H 5350 7250 50  0001 C CNN
+	1    5350 7250
+	1    0    0    -1
+$EndComp
+$Comp
+L -Mechanical:Fiducial FID2
+U 1 1 6051EF4F
+P 5850 7250
+F 0 "FID2" H 5935 7296 50  0000 L CNN
+F 1 "Fiducial" H 5935 7205 50  0000 L CNN
+F 2 "-Mechanical:Fiducial_1mm_Mask2mm" H 5850 7250 50  0001 C CNN
+F 3 "~" H 5850 7250 50  0001 C CNN
+	1    5850 7250
+	1    0    0    -1
+$EndComp
 $EndSCHEMATC

Commit message: update resistor values in enable line
Parts:
- R15: value 1k -> 10k; Desc 1kΩ ±5% 0.1W ±100ppm/℃ 0603 Chip Resistor - Surface Mount R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 -> 10kΩ ±5% 0.1W ±100ppm/℃ 0603 Chip Resistor - Surface Mount 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; LCSC# C14676 -> C99198; digikey# 311-1.0KGRTR-ND -> 311-10KGRTR-ND; element14# 9233385 -> 9233504; manf# RC0603JR-071KL -> RC0603JR-0710KL; mouser# 603-RC0603JR-071KL -> 603-RC0603JR-0710KL
- R18: value 10k -> 1k; Desc 10kΩ ±5% 0.1W ±100ppm/℃ 0603 Chip Resistor - Surface Mount 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 -> 1kΩ ±5% 0.1W ±100ppm/℃ 0603 Chip Resistor - Surface Mount R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; LCSC# C99198 -> C14676; digikey# 311-10KGRTR-ND -> 311-1.0KGRTR-ND; element14# 9233504 -> 9233385; manf# RC0603JR-0710KL -> RC0603JR-071KL; mouser# 603-RC0603JR-0710KL -> 603-RC0603JR-071KL
Changed lines of the file:
@@
 	8150 1750 8100 1750
-$Comp
-L -Passive:R R15
-U 1 1 60FED1B8
-P 8500 2900
-F 0 "R15" H 8350 2900 50  0000 C CNN
-F 1 "1k" V 8500 2900 50  0000 C CNN
-F 2 "-Passive:R_0603" V 8430 2900 50  0001 C CNN
-F 3 "https://www.yageo.com/upload/media/product/productsearch/datasheet/rchip/PYu-RC_Group_51_RoHS_L_11.pdf" H 8500 2900 50  0001 C CNN
-F 4 "1kΩ ±5% 0.1W ±100ppm/℃ 0603 Chip Resistor - Surface Mount RoHS" H 8500 2900 50  0001 C CNN "Desc"
-F 5 "Yageo" H 8500 2900 50  0001 C CNN "manf"
-F 6 "RC0603JR-071KL" H 8500 2900 50  0001 C CNN "manf#"
-F 7 "Yes" H 8500 2900 50  0001 C CNN "substitute"
-F 8 "C14676" H 8500 2900 50  0001 C CNN "LCSC#"
-F 9 "311-1.0KGRTR-ND" H 8500 2900 50  0001 C CNN "digikey#"
-F 10 "9233385" H 8500 2900 50  0001 C CNN "element14#"
-F 11 "603-RC0603JR-071KL" H 8500 2900 50  0001 C CNN "mouser#"
-	1    8500 2900
-	-1   0    0    1
-$EndComp
 $Comp
 L -Jumper:SolderJumper_2_Bridged_Alt JP8
@@
 Wire Wire Line
 	7300 5750 7250 5750
-$Comp
-L -Passive:R R18
-U 1 1 6044ADBA
-P 7550 2350
-F 0 "R18" V 7450 2350 50  0000 C CNN
-F 1 "10k" V 7550 2350 50  0000 C CNN
-F 2 "-Passive:R_0603" V 7480 2350 50  0001 L CNN
-F 3 "https://www.yageo.com/upload/media/product/productsearch/datasheet/rchip/PYu-RC_Group_51_RoHS_L_11.pdf" H 7550 2350 50  0001 L CNN
-F 4 "10kΩ ±5% 0.1W ±100ppm/℃ 0603 Chip Resistor - Surface Mount RoHS" H 7550 2350 50  0001 L CNN "Desc"
-F 5 "Yageo" H 7550 2350 50  0001 L CNN "manf"
-F 6 "RC0603JR-0710KL" H 7550 2350 50  0001 L CNN "manf#"
-F 7 "Yes" H 7550 2350 50  0001 L CNN "substitute"
-F 8 "C99198" H 7550 2350 50  0001 L CNN "LCSC#"
-F 9 "311-10KGRTR-ND" H 7550 2350 50  0001 L CNN "digikey#"
-F 10 "9233504" H 7550 2350 50  0001 L CNN "element14#"
-F 11 "603-RC0603JR-0710KL" H 7550 2350 50  0001 L CNN "mouser#"
-	1    7550 2350
-	0    1    1    0
-$EndComp
 Wire Wire Line
 	8100 2200 8100 2350
@@
 	1    0    0    -1
 $EndComp
+$Comp
+L -Passive:R R15
+U 1 1 60FED1B8
+P 8500 2900
+F 0 "R15" H 8350 2900 50  0000 C CNN
+F 1 "10k" V 8500 2900 50  0000 C CNN
+F 2 "-Passive:R_0603" V 8430 2900 50  0001 C CNN
+F 3 "https://www.yageo.com/upload/media/product/productsearch/datasheet/rchip/PYu-RC_Group_51_RoHS_L_11.pdf" H 8500 2900 50  0001 C CNN
+F 4 "10kΩ ±5% 0.1W ±100ppm/℃ 0603 Chip Resistor - Surface Mount RoHS" H 8500 2900 50  0001 C CNN "Desc"
+F 5 "Yageo" H 8500 2900 50  0001 C CNN "manf"
+F 6 "RC0603JR-0710KL" H 8500 2900 50  0001 C CNN "manf#"
+F 7 "Yes" H 8500 2900 50  0001 C CNN "substitute"
+F 8 "C99198" H 8500 2900 50  0001 C CNN "LCSC#"
+F 9 "311-10KGRTR-ND" H 8500 2900 50  0001 C CNN "digikey#"
+F 10 "9233504" H 8500 2900 50  0001 C CNN "element14#"
+F 11 "603-RC0603JR-0710KL" H 8500 2900 50  0001 C CNN "mouser#"
+	1    8500 2900
+	-1   0    0    1
+$EndComp
+$Comp
+L -Passive:R R18
+U 1 1 6044ADBA
+P 7550 2350
+F 0 "R18" V 7450 2350 50  0000 C CNN
+F 1 "1k" V 7550 2350 50  0000 C CNN
+F 2 "-Passive:R_0603" V 7480 2350 50  0001 L CNN
+F 3 "https://www.yageo.com/upload/media/product/productsearch/datasheet/rchip/PYu-RC_Group_51_RoHS_L_11.pdf" H 7550 2350 50  0001 L CNN
+F 4 "1kΩ ±5% 0.1W ±100ppm/℃ 0603 Chip Resistor - Surface Mount RoHS" H 7550 2350 50  0001 L CNN "Desc"
+F 5 "Yageo" H 7550 2350 50  0001 L CNN "manf"
+F 6 "RC0603JR-071KL" H 7550 2350 50  0001 L CNN "manf#"
+F 7 "Yes" H 7550 2350 50  0001 L CNN "substitute"
+F 8 "C14676" H 7550 2350 50  0001 L CNN "LCSC#"
+F 9 "311-1.0KGRTR-ND" H 7550 2350 50  0001 L CNN "digikey#"
+F 10 "9233385" H 7550 2350 50  0001 L CNN "element14#"
+F 11 "603-RC0603JR-071KL" H 7550 2350 50  0001 L CNN "mouser#"
+	1    7550 2350
+	0    1    1    0
+$EndComp
 $EndSCHEMATC

Commit message: remove breakout headers and simplify
Parts:
- removed C14: 0.1uF, -Passive:C_0603, symbol -Passive:C
- removed J3: Conn_01x08, -Connector:PinHeader_1x08_P2.54mm_Vertical_CBUS, symbol -Connector:Conn_01x08
- removed J4: Conn_01x06, -Connector:PinHeader_1x06_P2.54mm_Vertical_Arduino, symbol -Connector:Conn_01x06
- removed J5: Conn_01x08, -Connector:PinHeader_1x08_P2.54mm_Vertical_CTS, symbol -Connector:Conn_01x08
- removed JP1: SolderJumper_3_Bridged12, -Switch:SolderJumper-3_P1.3mm_Bridged12_RoundedPad1.0x1.5mm_NumberLabels, symbol -Jumper:SolderJumper_3_Bridged12
- removed JP2, JP3, JP4, JP5, JP6, JP7: SolderJumper_2_Bridged_Alt, -Switch:SolderJumper-2_P1.3mm_Bridged_RoundedPad1.0x1.5mm, symbol -Jumper:SolderJumper_2_Bridged_Alt
- removed Q3: 2N7002, -Chip:SOT-23-3, symbol -Discrete:2N7002
- removed R12, R16, R17: 1k, -Passive:R_0603, symbol -Passive:R
- removed R8, R9: 10k, -Passive:R_0603, symbol -Passive:R
- removed U6: NC7SZ66M5X, -Chip:SOT-23-5, symbol -Chip:NC7SZ66M5X
- added J4: Conn_01x04, -Connector:PinHeader_1x04_P2.54mm_Vertical_Arduino, symbol -Connector:Conn_01x04
Connections:
- net labels removed: +5V, CTS, DCD, DSR, DTR, RES, RI, RTS, SRES, VBUS, VOUT
- wire segments 213 -> 151
- no-connect marks 4 -> 10
Other:
- note removed: "Arduino Style Auto-Reset"
- note removed: "Cut trace on JP1 to switch\nVOUT from 5V to 3.3V"
- note removed: "Do not connect all three pads\non JP1 at the same time"
- moved on the sheet: C13

Commit message: change to larger tactile switch
Parts:
- removed SW1: B3U-1000P, -Switch:B3U-1000P, symbol -Switch:SW_MEC_5G
- added SW1: PTS810SJK250SMTRLFS, -Switch:PTS810SJK250SMTRLFS-TACT4.2MM, symbol -Switch:PTS810SJK250SMTRLFS
Connections:
- no-connect marks 10 -> 12
Changed lines of the file:
@@
-$EndComp
-$Comp
-L -Switch:SW_MEC_5G SW1
-U 1 1 603DC885
-P 7700 2800
-F 0 "SW1" V 7700 2700 50  0000 C CNN
-F 1 "B3U-1000P" H 7850 2700 50  0001 C CNN
-F 2 "-Switch:B3U-1000P" H 7700 3000 50  0001 L CNN
-F 3 "https://omronfs.omron.com/en_US/ecb/products/pdf/en-b3u.pdf" H 7700 3000 50  0001 L CNN
-F 4 "Tactile Switch SPST-NO Top Actuated Surface Mount" V 7700 2800 50  0001 L CNN "Desc"
-F 5 "Omron Electronics" V 7700 2800 50  0001 L CNN "manf"
-F 6 "B3U-1000P" V 7700 2800 50  0001 L CNN "manf#"
-F 7 "C231329" V 7700 2800 50  0001 L CNN "LCSC#"
-F 8 "SW1020CT-ND" V 7700 2800 50  0001 L CNN "digikey#"
-F 9 "1333652" V 7700 2800 50  0001 L CNN "element14#"
-F 10 "653-B3U-1000P" V 7700 2800 50  0001 L CNN "mouser#"
-	1    7700 2800
-	0    -1   1    0
 $EndComp
 $Comp
@@
 	5400 5150 5400 5100
 $Comp
-L -Flag:+3.3V #PWR?
+L -Flag:+3.3V #PWR0101
 U 1 1 60866490
 P 5050 1700
-F 0 "#PWR?" H 5050 1550 50  0001 C CNN
+F 0 "#PWR0101" H 5050 1550 50  0001 C CNN
 F 1 "+3.3V" H 5050 1850 50  0000 C CNN
 F 2 "" H 5050 1700 50  0001 C CNN
@@
 	1    0    0    -1
 $EndComp
+NoConn ~ 7750 2600
+NoConn ~ 7750 3000
+$Comp
+L -Switch:PTS810SJK250SMTRLFS SW1
+U 1 1 605F7932
+P 7700 2800
+F 0 "SW1" V 7700 3100 50  0000 R CNN
+F 1 "PTS810SJK250SMTRLFS" V 7655 2702 50  0001 R CNN
+F 2 "-Switch:PTS810SJK250SMTRLFS-TACT4.2MM" H 7700 3000 50  0001 C CNN
+F 3 "https://www.ckswitches.com/media/1476/pts810.pdf" H 7700 3000 50  0001 L CNN
+F 4 "SPST 50mA @ 16VDC Vertical Round Button SMD Tactile Switches RoHS" H 7250 2550 50  0001 L CNN "Desc"
+F 5 "C&K" H 7250 2450 50  0001 L CNN "manf"
+F 6 "PTS810SJK250SMTRLFS" H 7250 2350 50  0001 L CNN "manf#"
+F 7 "Yes" H 7250 2050 50  0001 L CNN "substitute"
+F 8 "C221896" H 7250 2150 50  0001 L CNN "LCSC#"
+F 9 "CKN10503TR-ND" H 7250 1950 50  0001 L CNN "digikey#"
+F 10 "3023215" H 7250 1850 50  0001 L CNN "element14#"
+F 11 "611-PTS810SJK250SMTR" H 7250 2250 50  0001 L CNN "mouser#"
+	1    7700 2800
+	0    -1   -1   0
+$EndComp
 $EndSCHEMATC
