File: hardware/kicad/ft231x_breakout_usb_power_switch/ft231x_breakout_usb_power_switch.kicad_pcb (KiCad board)
At the start: 2 copper layers, 60 x 31.2 mm, 50 parts, among them J1 USB_B_Micro_ALT, J2 USB_A_ALT, J3 Conn_01x08, J4 Conn_01x06, J5 Conn_01x08, Q3 2N7002, U1 SRV05-4, U2 FT231XS, U3 TPS2553DBVR, U4 SN74LVC1G04DBVR

Commit message: change footprint FT231XS to fix lcsc rotation filter
Parts:
- U2: footprint -Chip:FT231XS -> -Chip:SSOP-20_3.9x8.7mm_P0.635mm
Changed lines of the file:
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@@
     (add_net VBUS)
   )
-  (module -Chip:FT231XS (layer F.Cu)
+  (module -Chip:SSOP-20_3.9x8.7mm_P0.635mm (layer F.Cu)
     (at 132.8 84.8 270)
     (descr "SSOP20: plastic shrink small outline package; 24 leads; body width 3.9 mm; lead pitch 0.635; (see http://www.ftdichip.com/Support/Documents/DataSheets/ICs/DS_FT231X.pdf)")
     (tags "SSOP 0.635")
     (attr smd)
-    (fp_text reference U2 (at -2.05 -5.8 180) (layer F.SilkS)
+    (fp_text reference U2 (at -0.4 -5.8 180) (layer F.SilkS)
       (effects (font (size 0.8 0.8) (thickness 0.15)))
     )
-    (fp_text value FT231XS (at 0 5.4 90) (layer F.Fab) hide
+    (fp_text value FT231XS (at -0.3 -0.1 180) (layer F.Fab)
       (effects (font (size 1 1) (thickness 0.15)))
     )
-    (fp_text user %R (at 0 0 180) (layer F.Fab) hide
+    (fp_text user %R (at 0 0 90) (layer F.Fab)
       (effects (font (size 0.8 0.8) (thickness 0.15)))
     )

Commit message: Tidy up footprints and BoM fields
Parts:
- Q3: footprint -Chip:2N7002 -> -Chip:SOT-23-3
- U1: value SRV05-4 -> SOT-23-6; footprint -Chip:SRV05-4 -> -Chip:SOT-23-6
- U3: value TPS2553DBVR -> SOT-23-6; footprint -Chip:TPS2553DBVR -> -Chip:SOT-23-6
- U4: value SN74LVC1G04DBVR -> SOT-23-5; footprint -Chip:SN74LVC1G04DBVR -> -Chip:SOT-23-5
